File: ActuatorBoard.sch (KiCad schematic (older format))
At the start: 35 parts, among them J1 CONN_02X04, J2 Screw_Terminal_01x02, J3 Screw_Terminal_01x02, J4 CONN_02X04, J5 CONN_01X03, M1 Aktuator_Module, M2 Aktuator_Module, M3 Aktuator_Module, M4 Aktuator_Module, M5 Aktuator_Module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

Commit message: Changed position of two pins because of future h bridge pwm requirements
Connections:
- net SIG5: now also M2.6 (S1); no longer M2.3 (SIG)
- net SIG6: now also M2.3 (SIG); no longer M2.6 (S1)
Changed lines of the file:
@@
 Text GLabel 1250 800  2    60   Input ~ 0
 SIG4
+Text GLabel 2550 1000 2    60   Input ~ 0
+SIG5
 Text GLabel 2550 1200 2    60   Input ~ 0
-SIG5
-Text GLabel 2550 1000 2    60   Input ~ 0
 SIG6
 Text GLabel 2550 900  2    60   Input ~ 0

Commit message: Added actuator board drill and gerber
Connections:
- net SIG2: now also M2.6 (S1); no longer M1.6 (S1)
- net SIG5: now also M1.6 (S1); no longer M2.6 (S1)
Other:
- note added: "M1 - Module One\nSIG - D2 | S1 - D3 | S2 - D4 | S3 - D5 |\n\nM2 - Module Two\nSIG - D7 | S1 - D6 | S2 - D8 | S3 - D9 |\n\nM3 - Module Three\nSIG - D10 | S1 - D11 | S2 - D12 | S3 - A0 |\n\nM4 - Module Four\nSIG - A1 | S1 - A2 | S2 - A3 |\n\nM5 - Module Five\nSIG - A4\n\nM6 - Module Six\nSIG - A5"
- note removed: "M1 - Module One\nSIG - D2 | S1 - D3 | S2 - D4 | S3 - D5 |\n\nM2 - Module Two\nSIG - D6 | S1 - D7 | S2 - D8 | S3 - D9 |\n\nM3 - Module Three\nSIG - D10 | S1 - D11 | S2 - D12 | S3 - A0 |\n\nM4 - Module Four\nSIG - A1 | S1 - A2 | S2 - A3 |\n\nM5 - Module Five\nSIG - A4\n\nM6 - Module Six\nSIG - A5"
Changed lines of the file:
@@
 Text GLabel 1250 1200 2    60   Input ~ 0
 SIG1
-Text GLabel 1250 1000 2    60   Input ~ 0
+Text GLabel 2550 1000 2    60   Input ~ 0
 SIG2
 Text GLabel 1250 900  2    60   Input ~ 0
@@
 Text GLabel 1250 800  2    60   Input ~ 0
 SIG4
-Text GLabel 2550 1000 2    60   Input ~ 0
+Text GLabel 1250 1000 2    60   Input ~ 0
 SIG5
 Text GLabel 2550 1200 2    60   Input ~ 0
@@
 Arduino Nano
 Text Notes 9350 3650 0    118  ~ 0
-M1 - Module One\nSIG - D2 | S1 - D3 | S2 - D4 | S3 - D5 |\n\nM2 - Module Two\nSIG - D6 | S1 - D7 | S2 - D8 | S3 - D9 |\n\nM3 - Module Three\nSIG - D10 | S1 - D11 | S2 - D12 | S3 - A0 |\n\nM4 - Module Four\nSIG - A1 | S1 - A2 | S2 - A3 |\n\nM5 - Module Five\nSIG - A4\n\nM6 - Module Six\nSIG - A5
+M1 - Module One\nSIG - D2 | S1 - D3 | S2 - D4 | S3 - D5 |\n\nM2 - Module Two\nSIG - D7 | S1 - D6 | S2 - D8 | S3 - D9 |\n\nM3 - Module Three\nSIG - D10 | S1 - D11 | S2 - D12 | S3 - A0 |\n\nM4 - Module Four\nSIG - A1 | S1 - A2 | S2 - A3 |\n\nM5 - Module Five\nSIG - A4\n\nM6 - Module Six\nSIG - A5
 Wire Notes Line
 	9150 3750 14150 3750
